File: KiCAD/ZorroRAM.kicad_pcb (KiCad board)
At the start: 2 copper layers, 172.3 x 85.3 mm, 19 parts, among them J1 Conn_01x06_Male, U2 AP2210N-3.3TRG1, U3 74LVC245, U4 74LVC245, U5 XC9572XL-10VQ64C, U6 K4E641612D

Commit message: Add files via upload
Parts:
- moved C12 5.24 mm to (80.6, 121.0), turned to 90 degrees
Connections:
- ZorroSlot1 pad 1: Net-(ZorroSlot1-Pad1) -> GND
- ZorroSlot1 pad 3: Net-(ZorroSlot1-Pad3) -> GND
- ZorroSlot1 pad 99: Net-(ZorroSlot1-Pad99) -> GND
Routing:
- net GND: track 391.0 -> 83.7 mm, vias 6 -> 39
- net +3V3: track 321.6 -> 318.9 mm
- net /MD1: track 64.9 -> 66.2 mm
- net /_BUFOE: track 84.6 -> 85.6 mm
- added copper zone on B.Cu, net GND
- added copper zone on F.Cu, net GND
Other:
- board size 172.3 x 85.3 mm -> 129.1 x 85.3 mm
- net class Power: via_dia 1.3716 -> 0.8; via_drill 0.6096 -> 0.4
- board text added: "ZoRAM Amiga 2000 8 Megabyte Fast Ram Expansion Rev 0.7"
- board text added: "https://github.com/jasonsbeer/ZoRAM-Amiga-2000-RAM"
- board text removed: "ZoRAM Amiga 2000 8 Megabyte Fast Ram Expansion v 0.6 jasonsbeer https://github.com/jasonsbeer/ZoRAM-Amiga-2000-RAM Only AMIGA makes it possible."

Commit message: Add files via upload
Parts:
- added R1: 10k, Resistor_SMD:R_1206_3216Metric, F.Cu at (182.1, 138.4)
- moved C10 1.79 mm to (144.0, 81.5)
Routing:
- net /_CFGIN: track 47.7 -> 48.5 mm
- net +3V3: track 318.9 -> 318.2 mm
Other:
- board text added: "ZoRAM Amiga 2000 8 Megabyte Fast Ram Expansion Rev 0.8"
- board text removed: "ZoRAM Amiga 2000 8 Megabyte Fast Ram Expansion Rev 0.7"

Commit message: Add files via upload
Parts:
- removed R1: 10k, Resistor_SMD:R_1206_3216Metric
Routing:
- net /_CFGIN: track 48.5 -> 47.7 mm
- net GND: vias 39 -> 32
Other:
- board text added: "ZoRAM Amiga 2000 8 Megabyte Fast Ram Expansion Rev 0.7"
- board text removed: "ZoRAM Amiga 2000 8 Megabyte Fast Ram Expansion Rev 0.8"
